File: kicad/T1.kicad_pcb (KiCad board)
At the start: 2 copper layers, 311.9 x 145.3 mm, 168 parts, among them J1 USB_C_Receptacle, J2 AudioJack3, J3 AudioJack3, SW1 SW_Push, SW10 SW_Push, SW11 SW_Push, SW12 SW_Push, SW13 SW_Push, SW14 SW_Push, SW15 SW_Push, SW16 SW_Push, SW17 SW_Push, SW18 SW_Push, SW19 SW_Push, SW2 SW_Push, SW20 SW_Push, SW21 SW_Push, SW22 SW_Push, SW23 SW_Push, SW24 SW_Push, SW25 SW_Push, SW26 SW_Push, SW27 SW_Push, SW28 SW_Push, SW29 SW_Push, SW3 SW_Push, SW30 SW_Push, SW31 SW_Push, SW32 SW_Push, SW33 SW_Push, SW34 SW_Push, SW35 SW_Push, SW36 SW_Push, SW37 SW_Push, SW38 SW_Push, SW39 SW_Push, SW4 SW_Push, SW40 SW_Push, SW41 SW_Push, SW42 SW_Push, SW43 SW_Push, SW44 SW_Push, SW45 SW_Push, SW46 SW_Push, SW47 SW_Push, SW48 SW_Push, SW49 SW_Push, SW5 SW_Push, SW50 SW_Push, SW51 SW_Push, SW52 SW_Push, SW53 SW_Push, SW54 SW_Push, SW55 SW_Push, SW56 SW_Push, SW57 SW_Push, SW58 SW_Push, SW59 SW_Push, SW6 SW_Push, SW60 SW_Push, SW61 SW_Push, SW62 SW_Push, SW63 SW_Push, SW64 SW_Push, SW65 SW_Push, SW66 SW_Push, SW67 SW_Push, SW68 SW_Push, SW69 SW_Push, SW7 SW_Push, SW70 SW_Push, SW71 SW_Push, SW72 SW_Push, SW8 SW_Push, SW9 SW_Push, U1 ATmega32U4-AU, U2 ATmega32U4-AU, Y1 Crystal, Y2 Crystal

Commit message: main
Parts:
- added REF**: TestPoint_THTPad_1.0x1.0mm_Drill0.5mm, TestPoint:TestPoint_THTPad_1.0x1.0mm_Drill0.5mm, F.Cu at (186.9, 105.2)
- added REF**: chassi_mount_hole_4mm, panelization:chassi_mount_hole_4mm, F.Cu at (-12.7, 151.6)
- added REF**: TestPoint_THTPad_1.0x1.0mm_Drill0.5mm, TestPoint:TestPoint_THTPad_1.0x1.0mm_Drill0.5mm, F.Cu at (184.3, 105.2)
- added REF**: chassi_mount_hole_4mm, panelization:chassi_mount_hole_4mm, F.Cu at (290.5, 62.7)
- added REF**: chassi_mount_hole_4mm, panelization:chassi_mount_hole_4mm, F.Cu at (290.5, 151.6)
- added REF**: chassi_mount_hole_4mm, panelization:chassi_mount_hole_4mm, F.Cu at (158.8, 170.7)
- added REF**: chassi_mount_hole_4mm, panelization:chassi_mount_hole_4mm, F.Cu at (153.2, 61.1)
- added REF**: chassi_mount_hole_4mm, panelization:chassi_mount_hole_4mm, F.Cu at (124.6, 61.8)
- added REF**: chassi_mount_hole_4mm, panelization:chassi_mount_hole_4mm, F.Cu at (119.1, 170.7)
- added REF**: chassi_mount_hole_4mm, panelization:chassi_mount_hole_4mm, F.Cu at (-12.7, 62.5)
- moved J2 87.1 mm to (122.8, 137.5), turned to 190 degrees
- moved J3 87.1 mm to (154.9, 137.5), turned to 350 degrees
- moved C8 39.4 mm to (76.7, 106.6), turned to 45 degrees
- moved C7 36.2 mm to (69.5, 86.7), turned to 135 degrees
- moved R5 32.8 mm to (175.0, 87.5)
- moved C6 32.5 mm to (73.0, 82.9), turned to 315 degrees
- moved Y1 30.9 mm to (71.2, 84.8), turned to 135 degrees
- moved C11 24.7 mm to (175.1, 93.3), turned to 90 degrees
- moved R6 23.0 mm to (207.3, 89.9), turned to 270 degrees
- moved U2 21.4 mm to (189.4, 89.8), turned to 45 degrees
- moved U1 19.8 mm to (89.7, 90.3), turned to 45 degrees
- moved C10 19.7 mm to (181.7, 72.8), turned to 270 degrees
- moved R2 19.5 mm to (75.2, 91.3)
- moved R3 19.5 mm to (75.2, 88.9)
- moved C9 18.8 mm to (187.3, 72.8)
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Connections:
- Y1 pad 2: Net-(C6-Pad1) -> GND
- Y1 pad 3: (no net) -> Net-(C6-Pad1)
- Y1 pad 4: (no net) -> GND
- Y2 pad 2: Net-(C9-Pad1) -> Net-(C10-Pad2)
- Y2 pad 3: (no net) -> Net-(C9-Pad1)
- Y2 pad 4: (no net) -> Net-(C10-Pad2)
Routing:
- net Net-(C10-Pad2): track 89.8 -> 177.4 mm, vias 10 -> 13
- net VCC: track 116.1 -> 180.4 mm, vias 5 -> 4
- net Net-(J3-PadT): track 84.1 -> 133.4 mm
- net Net-(J3-PadR): track 35.4 -> 72.5 mm
- net Net-(J2-PadR): track 38.1 -> 68.6 mm, vias 1 -> 2
- net Net-(R5-Pad2): track 25.1 -> 54.3 mm, vias 1 -> 3
- net /rightButtonSheet/row4: track 180.8 -> 153.0 mm, vias 4 -> 2
- net Net-(R1-Pad2): track 27.9 -> 53.9 mm, vias 1 -> 3
- net /leftButtonSheet/row5: track 211.7 -> 187.4 mm
- net /rightButtonSheet/row5: track 209.7 -> 188.5 mm, vias 5 -> 2
- net /leftButtonSheet/row3: track 153.6 -> 133.5 mm, vias 1 -> 2
- net /leftButtonSheet/row4: track 181.5 -> 162.1 mm, vias 2 -> 1
- net /leftButtonSheet/row1: track 141.6 -> 159.3 mm, vias 2 -> 1
- net /leftButtonSheet/row2: track 136.5 -> 153.6 mm, vias 0 -> 1
- net GND: track 69.0 -> 52.0 mm, vias 11 -> 9
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- removed copper zone on B.Cu, net GND
- removed copper zone on B.Cu, net Net-(C10-Pad2)
Other:
- outline, holes or cut-outs redrawn
- board text added: "D+"
- board text added: "D-"
- board text added: "Fasth T1"
- board text added: "Jesper Fasth"
