File: kicad/T1.sch (KiCad schematic (older format))
At the start: 28 parts, among them J1 USB_C_Receptacle, J2 AudioJack3, J3 AudioJack3, SW36 SW_Push, SW37 SW_Push, U1 ATmega32U4-AU, U2 ATmega32U4-AU, Y1 Crystal, Y2 Crystal

Commit message: main
Connections:
- net GND: now also C1.1, C2.1, C3.1, C4.1, C5.1
Changed lines of the file:
@@
 Wire Wire Line
 	7000 2750 7100 2750
+$Comp
+L power:GND #PWR?
+U 1 1 611C34CC
+P 1600 3850
+F 0 "#PWR?" H 1600 3600 50  0001 C CNN
+F 1 "GND" H 1605 3677 50  0000 C CNN
+F 2 "" H 1600 3850 50  0001 C CNN
+F 3 "" H 1600 3850 50  0001 C CNN
+	1    1600 3850
+	-1   0    0    1
+$EndComp
+Wire Wire Line
+	1600 4100 1600 3850
+Connection ~ 1600 4100
 $EndSCHEMATC
