File: Schematic and pcb/T1.kicad_pcb (KiCad board)
At the start: 2 copper layers, 311.9 x 145.3 mm, 178 parts, among them J1 USB_C_Receptacle, J2 AudioJack3, J3 AudioJack3, SW1 SW_Push, SW10 SW_Push, SW11 SW_Push, SW12 SW_Push, SW13 SW_Push, SW14 SW_Push, SW15 SW_Push, SW16 SW_Push, SW17 SW_Push, SW18 SW_Push, SW19 SW_Push, SW2 SW_Push, SW20 SW_Push, SW21 SW_Push, SW22 SW_Push, SW23 SW_Push, SW24 SW_Push, SW25 SW_Push, SW26 SW_Push, SW27 SW_Push, SW28 SW_Push, SW29 SW_Push, SW3 SW_Push, SW30 SW_Push, SW31 SW_Push, SW32 SW_Push, SW33 SW_Push, SW34 SW_Push, SW35 SW_Push, SW36 SW_Push, SW37 SW_Push, SW38 SW_Push, SW39 SW_Push, SW4 SW_Push, SW40 SW_Push, SW41 SW_Push, SW42 SW_Push, SW43 SW_Push, SW44 SW_Push, SW45 SW_Push, SW46 SW_Push, SW47 SW_Push, SW48 SW_Push, SW49 SW_Push, SW5 SW_Push, SW50 SW_Push, SW51 SW_Push, SW52 SW_Push, SW53 SW_Push, SW54 SW_Push, SW55 SW_Push, SW56 SW_Push, SW57 SW_Push, SW58 SW_Push, SW59 SW_Push, SW6 SW_Push, SW60 SW_Push, SW61 SW_Push, SW62 SW_Push, SW63 SW_Push, SW64 SW_Push, SW65 SW_Push, SW66 SW_Push, SW67 SW_Push, SW68 SW_Push, SW69 SW_Push, SW7 SW_Push, SW70 SW_Push, SW71 SW_Push, SW72 SW_Push, SW8 SW_Push, SW9 SW_Push, U1 ATmega32U4-AU, U2 ATmega32U4-AU, Y1 Crystal, Y2 Crystal

Commit message: New pcb design
Parts:
- removed the REF** at (186.9, 105.2)
- removed the REF** at (-12.7, 151.6)
- removed the REF** at (184.3, 105.2)
- removed the REF** at (290.5, 62.7)
- removed the REF** at (290.5, 151.6)
- removed the REF** at (158.8, 170.7)
- removed the REF** at (153.2, 61.1)
- removed the REF** at (124.6, 61.8)
- removed the REF** at (119.1, 170.7)
- removed the REF** at (-12.7, 62.5)
- removed SW36, SW37: SW_Push, Button_Switch_THT:SW_PUSH_6mm
- added C12: 0.1u, Capacitor_SMD:C_1206_3216Metric, B.Cu at (162.1, 113.0)
- added D+: TestPoint, TestPoint:TestPoint_THTPad_1.0x1.0mm_Drill0.5mm, F.Cu at (140.5, 77.3)
- added D+: TestPoint, TestPoint:TestPoint_THTPad_1.0x1.0mm_Drill0.5mm, F.Cu at (158.7, 77.3)
- added D-: TestPoint, TestPoint:TestPoint_THTPad_1.0x1.0mm_Drill0.5mm, F.Cu at (140.5, 80.3)
- added D-: TestPoint, TestPoint:TestPoint_THTPad_1.0x1.0mm_Drill0.5mm, F.Cu at (158.7, 80.3)
- added REF**: MountingHole_2.2mm_M2_ISO7380, MountingHole:MountingHole_2.2mm_M2_ISO7380, F.Cu at (161.2, 128.8)
- added REF**: MountingHole_2.2mm_M2_ISO7380, MountingHole:MountingHole_2.2mm_M2_ISO7380, F.Cu at (159.4, 42.8)
- added REF**: KiCad-Logo2_5mm_SilkScreen, Symbol:KiCad-Logo2_5mm_SilkScreen, B.Cu at (260.0, 131.8)
- added REF**: KiCad-Logo2_5mm_SilkScreen, Symbol:KiCad-Logo2_5mm_SilkScreen, B.Cu at (39.3, 131.7)
- added REF**: OSHW-Logo2_7.3x6mm_SilkScreen, Symbol:OSHW-Logo2_7.3x6mm_SilkScreen, B.Cu at (270.9, 132.2)
- added REF**: OSHW-Logo2_7.3x6mm_SilkScreen, Symbol:OSHW-Logo2_7.3x6mm_SilkScreen, B.Cu at (27.7, 132.2)
- added REF**: MountingHole_2.2mm_M2_ISO7380, MountingHole:MountingHole_2.2mm_M2_ISO7380, F.Cu at (138.0, 128.9)
- added REF**: MountingHole_2.2mm_M2_ISO7380, MountingHole:MountingHole_2.2mm_M2_ISO7380, F.Cu at (296.9, 132.6)
- added REF**: MountingHole_2.2mm_M2_ISO7380, MountingHole:MountingHole_2.2mm_M2_ISO7380, F.Cu at (296.9, 43.7)
- added REF**: MountingHole_2.2mm_M2_ISO7380, MountingHole:MountingHole_2.2mm_M2_ISO7380, F.Cu at (2.38, 43.7)
- added REF**: MountingHole_2.2mm_M2_ISO7380, MountingHole:MountingHole_2.2mm_M2_ISO7380, F.Cu at (2.38, 132.6)
- added REF**: MountingHole_2.2mm_M2_ISO7380, MountingHole:MountingHole_2.2mm_M2_ISO7380, F.Cu at (165.2, 151.1)
- added REF**: MountingHole_2.2mm_M2_ISO7380, MountingHole:MountingHole_2.2mm_M2_ISO7380, F.Cu at (134.0, 151.1)
- added REF**: MountingHole_2.2mm_M2_ISO7380, MountingHole:MountingHole_2.2mm_M2_ISO7380, F.Cu at (139.9, 42.8)
- added TP1: TestPoint, TestPoint:TestPoint_THTPad_1.0x1.0mm_Drill0.5mm, F.Cu at (125.2, 35.7)
- added TP2: TestPoint, TestPoint:TestPoint_THTPad_1.0x1.0mm_Drill0.5mm, F.Cu at (125.2, 39.0)
- added TP3: TestPoint, TestPoint:TestPoint_THTPad_1.0x1.0mm_Drill0.5mm, F.Cu at (170.3, 38.7)
- added TP4: TestPoint, TestPoint:TestPoint_THTPad_1.0x1.0mm_Drill0.5mm, F.Cu at (160.1, 38.9)
- moved R3 62.3 mm to (135.7, 74.0)
- moved R2 62.1 mm to (135.7, 77.5)
- moved J1 33.1 mm to (132.6, 34.1)
- moved R8 33.1 mm to (131.1, 33.5)
- moved R7 33.1 mm to (133.8, 33.5)
- moved R5 31.5 mm to (176.2, 56.0), turned to 90 degrees
- moved C5 29.9 mm to (137.1, 57.8), turned to 270 degrees
- moved C8 26.0 mm to (96.7, 89.9)
- moved C4 25.1 mm to (134.2, 57.9), turned to 270 degrees
- moved R4 23.6 mm to (123.8, 72.8), turned to 270 degrees
- moved R1 22.6 mm to (92.5, 76.7), turned to 90 degrees
- moved J2 21.3 mm to (137.9, 122.4)
- moved D35 21.1 mm to (129.2, 132.7)
- moved D10 21.1 mm to (27.7, 123.9)
- moved D14 21.1 mm to (46.8, 101.3)
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Connections:
- C1 pad 1: Net-(C1-Pad1) -> GND
- C2 pad 1: Net-(C1-Pad1) -> GND
- C3 pad 1: Net-(C1-Pad1) -> GND
- C4 pad 1: Net-(C1-Pad1) -> GND
- C5 pad 1: Net-(C1-Pad1) -> GND
- J3 pad T: Net-(J3-PadT) -> Net-(C12-Pad2)
- R5 pad 1: Net-(J3-PadT) -> Net-(R5-Pad1)
- R5 pad 2: Net-(R5-Pad2) -> Net-(C12-Pad2)
- U1 pad 42: Net-(U1-Pad42) -> VCC
- U1 pad 8: Net-(U1-Pad8) -> VCC
- U2 pad 13: Net-(R5-Pad2) -> Net-(R5-Pad1)
- U2 pad 14: Net-(J3-PadT) -> Net-(C12-Pad2)
- U2 pad 2: Net-(J3-PadT) -> Net-(C12-Pad2)
- U2 pad 24: Net-(J3-PadT) -> Net-(C12-Pad2)
- U2 pad 34: Net-(J3-PadT) -> Net-(C12-Pad2)
- U2 pad 42: Net-(U2-Pad42) -> Net-(C12-Pad2)
- U2 pad 44: Net-(J3-PadT) -> Net-(C12-Pad2)
- U2 pad 7: Net-(J3-PadT) -> Net-(C12-Pad2)
Routing:
- net Net-(C12-Pad2): track 0.00 -> 156.2 mm, vias 0 -> 8
- net Net-(J3-PadT): track 133.4 -> 0.00 mm, vias 4 -> 0
- net /rightButtonSheet/column2: track 84.7 -> 139.1 mm
- net Net-(R5-Pad2): track 54.3 -> 0.00 mm, vias 3 -> 0
- net Net-(R5-Pad1): track 0.00 -> 49.6 mm
- net GND: track 52.0 -> 93.8 mm, vias 9 -> 17
- net Net-(R2-Pad1): track 13.7 -> 44.8 mm, vias 0 -> 2
- net Net-(TP6-Pad1): track 10.3 -> 38.5 mm, vias 1 -> 0
- net Net-(R3-Pad1): track 15.4 -> 43.0 mm, vias 0 -> 2
- net Net-(TP5-Pad1): track 12.1 -> 38.4 mm, vias 1 -> 0
- net /rightButtonSheet/column1: track 107.3 -> 130.8 mm
- net Net-(J3-PadR): track 72.5 -> 55.7 mm, vias 1 -> 0
- net /leftButtonSheet/row2: track 153.6 -> 137.3 mm, vias 1 -> 0
- net VCC: track 180.4 -> 196.3 mm, vias 4 -> 7
- net Net-(R1-Pad2): track 53.9 -> 69.7 mm, vias 3 -> 1
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- added copper zone on B.Cu, net GND
- added copper zone on B.Cu, net Net-(C10-Pad2)
Other:
- board size 311.9 x 145.3 mm -> 301.4 x 138.2 mm
- board text added: "@JesperFasth"
- board text added: "•"
- board text removed: "D+"
- board text removed: "D-"
- board text removed: "Jesper Fasth"

Commit message: Updated chassi base and removed key file
Parts:
- removed the D+ at (140.5, 77.3)
- removed the D+ at (158.7, 77.3)
- removed the D- at (140.5, 80.3)
- removed the D- at (158.7, 80.3)
- removed the REF** at (161.2, 128.8)
- removed the REF** at (159.4, 42.8)
- removed the REF** at (138.0, 128.9)
- removed the REF** at (296.9, 132.6)
- removed the REF** at (296.9, 43.7)
- removed the REF** at (2.38, 43.7)
- removed the REF** at (2.38, 132.6)
- removed the REF** at (165.2, 151.1)
- removed the REF** at (134.0, 151.1)
- removed the REF** at (139.9, 42.8)
- removed TP1, TP2, TP3, TP4: TestPoint, TestPoint:TestPoint_THTPad_1.0x1.0mm_Drill0.5mm
- added D+: TestPoint, TestPoint:TestPoint_THTPad_1.0x1.0mm_Drill0.5mm, F.Cu at (140.8, 77.3)
- added D+: TestPoint, TestPoint:TestPoint_THTPad_1.0x1.0mm_Drill0.5mm, F.Cu at (159.0, 77.3)
- added D-: TestPoint, TestPoint:TestPoint_THTPad_1.0x1.0mm_Drill0.5mm, F.Cu at (140.8, 80.3)
- added D-: TestPoint, TestPoint:TestPoint_THTPad_1.0x1.0mm_Drill0.5mm, F.Cu at (159.0, 80.3)
- added GND: TestPoint, TestPoint:TestPoint_THTPad_1.0x1.0mm_Drill0.5mm, F.Cu at (125.4, 35.7)
- added GND: TestPoint, TestPoint:TestPoint_THTPad_1.0x1.0mm_Drill0.5mm, F.Cu at (170.5, 38.7)
- added REF**: MountingHole_2.2mm_M2_ISO7380, MountingHole:MountingHole_2.2mm_M2_ISO7380, F.Cu at (161.4, 128.8)
- added REF**: MountingHole_2.2mm_M2_ISO7380, MountingHole:MountingHole_2.2mm_M2_ISO7380, F.Cu at (159.6, 42.8)
- added REF**: MountingHole_2.2mm_M2_ISO7380, MountingHole:MountingHole_2.2mm_M2_ISO7380, F.Cu at (138.3, 128.9)
- added REF**: MountingHole_2.2mm_M2_ISO7380, MountingHole:MountingHole_2.2mm_M2_ISO7380, F.Cu at (297.1, 132.5)
- added REF**: MountingHole_2.2mm_M2_ISO7380, MountingHole:MountingHole_2.2mm_M2_ISO7380, F.Cu at (297.1, 43.6)
- added REF**: MountingHole_2.2mm_M2_ISO7380, MountingHole:MountingHole_2.2mm_M2_ISO7380, F.Cu at (2.65, 43.6)
- added REF**: MountingHole_2.2mm_M2_ISO7380, MountingHole:MountingHole_2.2mm_M2_ISO7380, F.Cu at (2.65, 132.5)
- added REF**: MountingHole_2.2mm_M2_ISO7380, MountingHole:MountingHole_2.2mm_M2_ISO7380, F.Cu at (165.5, 151.1)
- added REF**: MountingHole_2.2mm_M2_ISO7380, MountingHole:MountingHole_2.2mm_M2_ISO7380, F.Cu at (134.3, 151.1)
- added REF**: MountingHole_2.2mm_M2_ISO7380, MountingHole:MountingHole_2.2mm_M2_ISO7380, F.Cu at (140.2, 42.8)
- added RESET: TestPoint, TestPoint:TestPoint_THTPad_1.0x1.0mm_Drill0.5mm, F.Cu at (125.4, 39.0)
- added RESET: TestPoint, TestPoint:TestPoint_THTPad_1.0x1.0mm_Drill0.5mm, F.Cu at (160.4, 38.9)
- moved SW68 0.27 mm to (288.7, 45.1)
- moved SW70 0.27 mm to (288.7, 83.2)
- moved SW71 0.27 mm to (288.7, 102.3)
- moved SW72 0.27 mm to (288.7, 121.3)
- moved SW69 0.27 mm to (288.7, 64.2)
- moved D52 0.27 mm to (233.7, 60.2)
- moved D54 0.27 mm to (233.7, 98.3)
- moved D55 0.27 mm to (233.7, 117.4)
- moved R7 0.27 mm to (134.1, 33.5)
- moved Y2 0.27 mm to (194.9, 56.6)
- moved C9 0.27 mm to (198.4, 56.8)
- moved D31 0.27 mm to (123.2, 47.6)
- moved D32 0.27 mm to (123.2, 66.7)
- moved R1 0.27 mm to (92.8, 76.7)
- moved SW26 0.27 mm to (116.3, 43.4)
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Connections:
- U1 pad 42: VCC -> Net-(U1-Pad42)
- U2 pad 42: Net-(C12-Pad2) -> Net-(U2-Pad42)
- U2 pad 8: Net-(U2-Pad8) -> Net-(C10-Pad2)
Routing:
- net Net-(C10-Pad2): track 183.4 -> 193.9 mm
- net VCC: track 196.3 -> 194.6 mm
- net Net-(C12-Pad2): track 156.2 -> 155.2 mm
Other:
- outline, holes or cut-outs redrawn
