File: Schematic and pcb/T1.sch (KiCad schematic (older format))
At the start: 28 parts, among them J1 USB_C_Receptacle, J2 AudioJack3, J3 AudioJack3, SW36 SW_Push, SW37 SW_Push, U1 ATmega32U4-AU, U2 ATmega32U4-AU, Y1 Crystal, Y2 Crystal

Commit message: New pcb design
Parts:
- removed SW36, SW37: SW_Push, Button_Switch_THT:SW_PUSH_6mm, symbol Switch:SW_Push
- added C12: 0.1u, Capacitor_SMD:C_1206_3216Metric, symbol Device:C_Small
- added TP1, TP2, TP3, TP4, TP5, TP6, TP7, TP8: TestPoint, TestPoint:TestPoint_THTPad_1.0x1.0mm_Drill0.5mm, symbol Connector:TestPoint
Connections:
- net GND: now also TP1.1
- net VCC: now also U1.42 (AREF), U1.8 (PB0)
- net at C10.2, C11.1, C9.2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: now also C12.1, TP3.1
- net at J3.T, U2.14 (VCC), U2.2 (UVCC)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: now also R5.2, U2.42 (AREF), C12.2; no longer R5.1
- net at R1.2, U1.13 (~RESET): now also TP2.1
- net at R2.1, U1.3 (D-): now also TP7.1
- net at R3.1, U1.4 (D+): now also TP8.1
- net at U2.13 (~RESET): now also R5.1, TP4.1; no longer R5.2
- net at U2.3 (D-): now also TP6.1
- net at U2.4 (D+): now also TP5.1
Other:
- moved on the sheet: C1, C2, C3, C4, C5, J2, R2, R3, R5

Commit message: Updated chassi base and removed key file
Connections:
- net VCC: no longer U1.42 (AREF)
- net at C10.2, C11.1, C12.1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: now also U2.8 (PB0)
- net at C12.2, J3.T, R5.2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: no longer U2.42 (AREF)
Changed lines of the file:
@@
 	0    -1   -1   0
-$EndComp
-Connection ~ 3150 1100
-Wire Wire Line
-	3150 1100 3250 1100
-Connection ~ 3050 1100
-Wire Wire Line
-	3050 1100 3150 1100
-Wire Wire Line
-	3050 1100 2950 1100
-$Comp
-L MCU_Microchip_ATmega:ATmega32U4-AU U1
-U 1 1 61114792
-P 3150 2900
-F 0 "U1" H 3150 1011 50  0000 C CNN
-F 1 "ATmega32U4-AU" H 3150 920 50  0000 C CNN
-F 2 "Package_QFP:TQFP-44_10x10mm_P0.8mm" H 3150 2900 50  0001 C CIN
-F 3 "http://ww1.microchip.com/downloads/en/DeviceDoc/Atmel-7766-8-bit-AVR-ATmega16U4-32U4_Datasheet.pdf" H 3150 2900 50  0001 C CNN
-	1    3150 2900
-	1    0    0    -1
 $EndComp
 $Comp
@@
 Wire Wire Line
 	3050 4700 3150 4700
-Connection ~ 3150 4700
 $Comp
 L power:VCC #PWR08
@@
 Wire Wire Line
 	2500 4850 2500 5350
-Wire Wire Line
-	2550 2000 2550 2200
-Connection ~ 2550 2200
-Wire Wire Line
-	7300 2050 7300 2250
-Connection ~ 7300 2250
 $Comp
 L Device:C_Small C12
@@
 Wire Wire Line
 	7800 3800 7800 4750
+Wire Wire Line
+	3050 1100 2950 1100
+Connection ~ 3050 1100
+Connection ~ 3150 4700
+Wire Wire Line
+	3050 1100 3150 1100
+Wire Wire Line
+	3150 1100 3250 1100
+Connection ~ 3150 1100
+$Comp
+L MCU_Microchip_ATmega:ATmega32U4-AU U1
+U 1 1 61114792
+P 3150 2900
+F 0 "U1" H 3150 1011 50  0000 C CNN
+F 1 "ATmega32U4-AU" H 3150 920 50  0000 C CNN
+F 2 "Package_QFP:TQFP-44_10x10mm_P0.8mm" H 3150 2900 50  0001 C CIN
+F 3 "http://ww1.microchip.com/downloads/en/DeviceDoc/Atmel-7766-8-bit-AVR-ATmega16U4-32U4_Datasheet.pdf" H 3150 2900 50  0001 C CNN
+	1    3150 2900
+	1    0    0    -1
+$EndComp
+Wire Wire Line
+	8500 1450 7800 1450
+Wire Wire Line
+	7800 1450 7800 3300
+Connection ~ 7800 3300
 $EndSCHEMATC
