File: Schematic and pcb/xenophon.sch (KiCad schematic (older format))
At the start: 35 parts, among them J1 USB_C_Receptacle, J2 AudioJack3, J3 AudioJack3, U1 ATmega32U4-AU, U2 ATmega32U4-AU, Y1 Crystal, Y2 Crystal

Commit message: Changed name
Changed lines of the file:
@@
 U 6107657D
 F0 "leftButtonSheet" 50
-F1 "file6107657C.sch" 50
+F1 "leftButtonSheet.sch" 50
 F2 "row1" I L 4800 1950 50
 F3 "row2" I L 4800 2050 50
@@
 U 6116737E
 F0 "rightButtonSheet" 50
-F1 "file6116737D.sch" 50
+F1 "rightButtonSheet.sch" 50
 F2 "row1" I L 9550 2000 50
 F3 "row2" I L 9550 2100 50
