File: Schematic and pcb/leftButtonSheet.sch (KiCad schematic (older format))
At the start: 70 parts, among them SW1 SW_Push, SW10 SW_Push, SW11 SW_Push, SW12 SW_Push, SW13 SW_Push, SW14 SW_Push, SW15 SW_Push, SW16 SW_Push, SW17 SW_Push, SW18 SW_Push, SW19 SW_Push, SW2 SW_Push, SW20 SW_Push, SW21 SW_Push, SW22 SW_Push, SW23 SW_Push, SW24 SW_Push, SW25 SW_Push, SW26 SW_Push, SW27 SW_Push, SW28 SW_Push, SW29 SW_Push, SW3 SW_Push, SW30 SW_Push, SW31 SW_Push, SW32 SW_Push, SW33 SW_Push, SW34 SW_Push, SW35 SW_Push, SW4 SW_Push, SW5 SW_Push, SW6 SW_Push, SW7 SW_Push, SW8 SW_Push, SW9 SW_Push

Commit message: Updated pcb and projekt files.
Parts:
- SW1, SW2, SW3, SW4, SW5: footprint keyswitch:SW_Cherry_MX_1.50u_PCB -> XenophonFootprintLibrary:SW_Cherry_MX_1.50u_PCB
- SW10, SW11, SW12, SW13, SW14, SW15, SW16, SW17, SW18, SW19, SW20, SW21, SW22, SW23, SW24, SW25, SW26, SW27, SW28, SW29, SW30, SW31, SW32, SW33, SW34, SW35, SW6, SW7, SW8, SW9: footprint keyswitch:SW_Cherry_MX_1.00u_PCB -> XenophonFootprintLibrary:SW_Cherry_MX_1.00u_PCB
Changed lines of the file:
@@
 F 0 "SW1" H 1950 2485 50  0000 C CNN
 F 1 "SW_Push" H 1950 2394 50  0000 C CNN
-F 2 "keyswitch:SW_Cherry_MX_1.50u_PCB" H 1950 2400 50  0001 C CNN
+F 2 "XenophonFootprintLibrary:SW_Cherry_MX_1.50u_PCB" H 1950 2400 50  0001 C CNN
 F 3 "~" H 1950 2400 50  0001 C CNN
 	1    1950 2200
@@
 F 0 "SW2" H 1950 2935 50  0000 C CNN
 F 1 "SW_Push" H 1950 2844 50  0000 C CNN
-F 2 "keyswitch:SW_Cherry_MX_1.50u_PCB" H 1950 2850 50  0001 C CNN
+F 2 "XenophonFootprintLibrary:SW_Cherry_MX_1.50u_PCB" H 1950 2850 50  0001 C CNN
 F 3 "~" H 1950 2850 50  0001 C CNN
 	1    1950 2650
@@
 F 0 "SW3" H 1950 3385 50  0000 C CNN
 F 1 "SW_Push" H 1950 3294 50  0000 C CNN
-F 2 "keyswitch:SW_Cherry_MX_1.50u_PCB" H 1950 3300 50  0001 C CNN
+F 2 "XenophonFootprintLibrary:SW_Cherry_MX_1.50u_PCB" H 1950 3300 50  0001 C CNN
 F 3 "~" H 1950 3300 50  0001 C CNN
 	1    1950 3100
@@
 F 0 "SW4" H 1950 3835 50  0000 C CNN
 F 1 "SW_Push" H 1950 3744 50  0000 C CNN
-F 2 "keyswitch:SW_Cherry_MX_1.50u_PCB" H 1950 3750 50  0001 C CNN
+F 2 "XenophonFootprintLibrary:SW_Cherry_MX_1.50u_PCB" H 1950 3750 50  0001 C CNN
 F 3 "~" H 1950 3750 50  0001 C CNN
 	1    1950 3550
@@
 F 0 "SW5" H 1950 4285 50  0000 C CNN
 F 1 "SW_Push" H 1950 4194 50  0000 C CNN
-F 2 "keyswitch:SW_Cherry_MX_1.50u_PCB" H 1950 4200 50  0001 C CNN
+F 2 "XenophonFootprintLibrary:SW_Cherry_MX_1.50u_PCB" H 1950 4200 50  0001 C CNN
 F 3 "~" H 1950 4200 50  0001 C CNN
 	1    1950 4000
@@
 F 0 "SW6" H 2850 2485 50  0000 C CNN
 F 1 "SW_Push" H 2850 2394 50  0000 C CNN
-F 2 "keyswitch:SW_Cherry_MX_1.00u_PCB" H 2850 2400 50  0001 C CNN
+F 2 "XenophonFootprintLibrary:SW_Cherry_MX_1.00u_PCB" H 2850 2400 50  0001 C CNN
 F 3 "~" H 2850 2400 50  0001 C CNN
 	1    2850 2200
@@
 F 0 "SW7" H 2850 2935 50  0000 C CNN
 F 1 "SW_Push" H 2850 2844 50  0000 C CNN
-F 2 "keyswitch:SW_Cherry_MX_1.00u_PCB" H 2850 2850 50  0001 C CNN
+F 2 "XenophonFootprintLibrary:SW_Cherry_MX_1.00u_PCB" H 2850 2850 50  0001 C CNN
 F 3 "~" H 2850 2850 50  0001 C CNN
 	1    2850 2650
@@
 F 0 "SW8" H 2850 3385 50  0000 C CNN
 F 1 "SW_Push" H 2850 3294 50  0000 C CNN
-F 2 "keyswitch:SW_Cherry_MX_1.00u_PCB" H 2850 3300 50  0001 C CNN
+F 2 "XenophonFootprintLibrary:SW_Cherry_MX_1.00u_PCB" H 2850 3300 50  0001 C CNN
 F 3 "~" H 2850 3300 50  0001 C CNN
 	1    2850 3100
@@
 F 0 "SW9" H 2850 3835 50  0000 C CNN
 F 1 "SW_Push" H 2850 3744 50  0000 C CNN
-F 2 "keyswitch:SW_Cherry_MX_1.00u_PCB" H 2850 3750 50  0001 C CNN
+F 2 "XenophonFootprintLibrary:SW_Cherry_MX_1.00u_PCB" H 2850 3750 50  0001 C CNN
 F 3 "~" H 2850 3750 50  0001 C CNN
 	1    2850 3550
@@
 F 0 "SW10" H 2850 4285 50  0000 C CNN
 F 1 "SW_Push" H 2850 4194 50  0000 C CNN
-F 2 "keyswitch:SW_Cherry_MX_1.00u_PCB" H 2850 4200 50  0001 C CNN
+F 2 "XenophonFootprintLibrary:SW_Cherry_MX_1.00u_PCB" H 2850 4200 50  0001 C CNN
 F 3 "~" H 2850 4200 50  0001 C CNN
 	1    2850 4000
@@
 F 0 "SW11" H 3750 2485 50  0000 C CNN
 F 1 "SW_Push" H 3750 2394 50  0000 C CNN
-F 2 "keyswitch:SW_Cherry_MX_1.00u_PCB" H 3750 2400 50  0001 C CNN
+F 2 "XenophonFootprintLibrary:SW_Cherry_MX_1.00u_PCB" H 3750 2400 50  0001 C CNN
 F 3 "~" H 3750 2400 50  0001 C CNN
 	1    3750 2200
@@
 F 0 "SW12" H 3750 2935 50  0000 C CNN
 F 1 "SW_Push" H 3750 2844 50  0000 C CNN
-F 2 "keyswitch:SW_Cherry_MX_1.00u_PCB" H 3750 2850 50  0001 C CNN
+F 2 "XenophonFootprintLibrary:SW_Cherry_MX_1.00u_PCB" H 3750 2850 50  0001 C CNN
 F 3 "~" H 3750 2850 50  0001 C CNN
 	1    3750 2650
@@
 F 0 "SW13" H 3750 3385 50  0000 C CNN
 F 1 "SW_Push" H 3750 3294 50  0000 C CNN
-F 2 "keyswitch:SW_Cherry_MX_1.00u_PCB" H 3750 3300 50  0001 C CNN
+F 2 "XenophonFootprintLibrary:SW_Cherry_MX_1.00u_PCB" H 3750 3300 50  0001 C CNN
 F 3 "~" H 3750 3300 50  0001 C CNN
 	1    3750 3100
@@
 F 0 "SW14" H 3750 3835 50  0000 C CNN
 F 1 "SW_Push" H 3750 3744 50  0000 C CNN
-F 2 "keyswitch:SW_Cherry_MX_1.00u_PCB" H 3750 3750 50  0001 C CNN
+F 2 "XenophonFootprintLibrary:SW_Cherry_MX_1.00u_PCB" H 3750 3750 50  0001 C CNN
 F 3 "~" H 3750 3750 50  0001 C CNN
 	1    3750 3550
@@
 F 0 "SW15" H 3750 4285 50  0000 C CNN
 F 1 "SW_Push" H 3750 4194 50  0000 C CNN
-F 2 "keyswitch:SW_Cherry_MX_1.00u_PCB" H 3750 4200 50  0001 C CNN
+F 2 "XenophonFootprintLibrary:SW_Cherry_MX_1.00u_PCB" H 3750 4200 50  0001 C CNN
 F 3 "~" H 3750 4200 50  0001 C CNN
 	1    3750 4000
@@
 F 0 "SW16" H 4650 2485 50  0000 C CNN
 F 1 "SW_Push" H 4650 2394 50  0000 C CNN
-F 2 "keyswitch:SW_Cherry_MX_1.00u_PCB" H 4650 2400 50  0001 C CNN
+F 2 "XenophonFootprintLibrary:SW_Cherry_MX_1.00u_PCB" H 4650 2400 50  0001 C CNN
 F 3 "~" H 4650 2400 50  0001 C CNN
 	1    4650 2200
@@
 F 0 "SW17" H 4650 2935 50  0000 C CNN
 F 1 "SW_Push" H 4650 2844 50  0000 C CNN
-F 2 "keyswitch:SW_Cherry_MX_1.00u_PCB" H 4650 2850 50  0001 C CNN
+F 2 "XenophonFootprintLibrary:SW_Cherry_MX_1.00u_PCB" H 4650 2850 50  0001 C CNN
 F 3 "~" H 4650 2850 50  0001 C CNN
 	1    4650 2650
@@
 F 0 "SW18" H 4650 3385 50  0000 C CNN
 F 1 "SW_Push" H 4650 3294 50  0000 C CNN
-F 2 "keyswitch:SW_Cherry_MX_1.00u_PCB" H 4650 3300 50  0001 C CNN
+F 2 "XenophonFootprintLibrary:SW_Cherry_MX_1.00u_PCB" H 4650 3300 50  0001 C CNN
 F 3 "~" H 4650 3300 50  0001 C CNN
 	1    4650 3100
@@
 F 0 "SW19" H 4650 3835 50  0000 C CNN
 F 1 "SW_Push" H 4650 3744 50  0000 C CNN
-F 2 "keyswitch:SW_Cherry_MX_1.00u_PCB" H 4650 3750 50  0001 C CNN
+F 2 "XenophonFootprintLibrary:SW_Cherry_MX_1.00u_PCB" H 4650 3750 50  0001 C CNN
 F 3 "~" H 4650 3750 50  0001 C CNN
 	1    4650 3550
@@
 F 0 "SW20" H 4650 4285 50  0000 C CNN
 F 1 "SW_Push" H 4650 4194 50  0000 C CNN
-F 2 "keyswitch:SW_Cherry_MX_1.00u_PCB" H 4650 4200 50  0001 C CNN
+F 2 "XenophonFootprintLibrary:SW_Cherry_MX_1.00u_PCB" H 4650 4200 50  0001 C CNN
 F 3 "~" H 4650 4200 50  0001 C CNN
 	1    4650 4000
@@
 F 0 "SW21" H 5550 2485 50  0000 C CNN
 F 1 "SW_Push" H 5550 2394 50  0000 C CNN
-F 2 "keyswitch:SW_Cherry_MX_1.00u_PCB" H 5550 2400 50  0001 C CNN
+F 2 "XenophonFootprintLibrary:SW_Cherry_MX_1.00u_PCB" H 5550 2400 50  0001 C CNN
 F 3 "~" H 5550 2400 50  0001 C CNN
 	1    5550 2200
@@
 F 0 "SW22" H 5550 2935 50  0000 C CNN
 F 1 "SW_Push" H 5550 2844 50  0000 C CNN
-F 2 "keyswitch:SW_Cherry_MX_1.00u_PCB" H 5550 2850 50  0001 C CNN
+F 2 "XenophonFootprintLibrary:SW_Cherry_MX_1.00u_PCB" H 5550 2850 50  0001 C CNN
 F 3 "~" H 5550 2850 50  0001 C CNN
 	1    5550 2650
@@
 F 0 "SW23" H 5550 3385 50  0000 C CNN
 F 1 "SW_Push" H 5550 3294 50  0000 C CNN
-F 2 "keyswitch:SW_Cherry_MX_1.00u_PCB" H 5550 3300 50  0001 C CNN
+F 2 "XenophonFootprintLibrary:SW_Cherry_MX_1.00u_PCB" H 5550 3300 50  0001 C CNN
 F 3 "~" H 5550 3300 50  0001 C CNN
 	1    5550 3100
@@
 F 0 "SW24" H 5550 3835 50  0000 C CNN
 F 1 "SW_Push" H 5550 3744 50  0000 C CNN
-F 2 "keyswitch:SW_Cherry_MX_1.00u_PCB" H 5550 3750 50  0001 C CNN
+F 2 "XenophonFootprintLibrary:SW_Cherry_MX_1.00u_PCB" H 5550 3750 50  0001 C CNN
 F 3 "~" H 5550 3750 50  0001 C CNN
 	1    5550 3550
@@
 F 0 "SW25" H 5550 4285 50  0000 C CNN
 F 1 "SW_Push" H 5550 4194 50  0000 C CNN
-F 2 "keyswitch:SW_Cherry_MX_1.00u_PCB" H 5550 4200 50  0001 C CNN
+F 2 "XenophonFootprintLibrary:SW_Cherry_MX_1.00u_PCB" H 5550 4200 50  0001 C CNN
 F 3 "~" H 5550 4200 50  0001 C CNN
 	1    5550 4000
@@
 F 0 "SW26" H 6450 2485 50  0000 C CNN
 F 1 "SW_Push" H 6450 2394 50  0000 C CNN
-F 2 "keyswitch:SW_Cherry_MX_1.00u_PCB" H 6450 2400 50  0001 C CNN
+F 2 "XenophonFootprintLibrary:SW_Cherry_MX_1.00u_PCB" H 6450 2400 50  0001 C CNN
 F 3 "~" H 6450 2400 50  0001 C CNN
 	1    6450 2200
@@
 F 0 "SW27" H 6450 2935 50  0000 C CNN
 F 1 "SW_Push" H 6450 2844 50  0000 C CNN
-F 2 "keyswitch:SW_Cherry_MX_1.00u_PCB" H 6450 2850 50  0001 C CNN
+F 2 "XenophonFootprintLibrary:SW_Cherry_MX_1.00u_PCB" H 6450 2850 50  0001 C CNN
 F 3 "~" H 6450 2850 50  0001 C CNN
 	1    6450 2650
@@
 F 0 "SW28" H 6450 3385 50  0000 C CNN
 F 1 "SW_Push" H 6450 3294 50  0000 C CNN
-F 2 "keyswitch:SW_Cherry_MX_1.00u_PCB" H 6450 3300 50  0001 C CNN
+F 2 "XenophonFootprintLibrary:SW_Cherry_MX_1.00u_PCB" H 6450 3300 50  0001 C CNN
 F 3 "~" H 6450 3300 50  0001 C CNN
 	1    6450 3100
@@
 F 0 "SW29" H 6450 3835 50  0000 C CNN
 F 1 "SW_Push" H 6450 3744 50  0000 C CNN
-F 2 "keyswitch:SW_Cherry_MX_1.00u_PCB" H 6450 3750 50  0001 C CNN
+F 2 "XenophonFootprintLibrary:SW_Cherry_MX_1.00u_PCB" H 6450 3750 50  0001 C CNN
 F 3 "~" H 6450 3750 50  0001 C CNN
 	1    6450 3550
@@
 F 0 "SW30" H 6450 4285 50  0000 C CNN
 F 1 "SW_Push" H 6450 4194 50  0000 C CNN
-F 2 "keyswitch:SW_Cherry_MX_1.00u_PCB" H 6450 4200 50  0001 C CNN
+F 2 "XenophonFootprintLibrary:SW_Cherry_MX_1.00u_PCB" H 6450 4200 50  0001 C CNN
 F 3 "~" H 6450 4200 50  0001 C CNN
 	1    6450 4000
@@
 F 0 "SW31" H 7350 2485 50  0000 C CNN
 F 1 "SW_Push" H 7350 2394 50  0000 C CNN
-F 2 "keyswitch:SW_Cherry_MX_1.00u_PCB" H 7350 2400 50  0001 C CNN
+F 2 "XenophonFootprintLibrary:SW_Cherry_MX_1.00u_PCB" H 7350 2400 50  0001 C CNN
 F 3 "~" H 7350 2400 50  0001 C CNN
 	1    7350 2200
@@
 F 0 "SW32" H 7350 2935 50  0000 C CNN
 F 1 "SW_Push" H 7350 2844 50  0000 C CNN
-F 2 "keyswitch:SW_Cherry_MX_1.00u_PCB" H 7350 2850 50  0001 C CNN
+F 2 "XenophonFootprintLibrary:SW_Cherry_MX_1.00u_PCB" H 7350 2850 50  0001 C CNN
 F 3 "~" H 7350 2850 50  0001 C CNN
 	1    7350 2650
@@
 F 0 "SW33" H 7350 3385 50  0000 C CNN
 F 1 "SW_Push" H 7350 3294 50  0000 C CNN
-F 2 "keyswitch:SW_Cherry_MX_1.00u_PCB" H 7350 3300 50  0001 C CNN
+F 2 "XenophonFootprintLibrary:SW_Cherry_MX_1.00u_PCB" H 7350 3300 50  0001 C CNN
 F 3 "~" H 7350 3300 50  0001 C CNN
 	1    7350 3100
@@
 F 0 "SW34" H 7350 3835 50  0000 C CNN
 F 1 "SW_Push" H 7350 3744 50  0000 C CNN
-F 2 "keyswitch:SW_Cherry_MX_1.00u_PCB" H 7350 3750 50  0001 C CNN
+F 2 "XenophonFootprintLibrary:SW_Cherry_MX_1.00u_PCB" H 7350 3750 50  0001 C CNN
 F 3 "~" H 7350 3750 50  0001 C CNN
 	1    7350 3550
@@
 F 0 "SW35" H 7350 4285 50  0000 C CNN
 F 1 "SW_Push" H 7350 4194 50  0000 C CNN
-F 2 "keyswitch:SW_Cherry_MX_1.00u_PCB" H 7350 4200 50  0001 C CNN
+F 2 "XenophonFootprintLibrary:SW_Cherry_MX_1.00u_PCB" H 7350 4200 50  0001 C CNN
 F 3 "~" H 7350 4200 50  0001 C CNN
 	1    7350 4000
