File: Schematic and pcb/rightButtonSheet.sch (KiCad schematic (older format))
At the start: 70 parts, among them SW38 SW_Push, SW39 SW_Push, SW40 SW_Push, SW41 SW_Push, SW42 SW_Push, SW43 SW_Push, SW44 SW_Push, SW45 SW_Push, SW46 SW_Push, SW47 SW_Push, SW48 SW_Push, SW49 SW_Push, SW50 SW_Push, SW51 SW_Push, SW52 SW_Push, SW53 SW_Push, SW54 SW_Push, SW55 SW_Push, SW56 SW_Push, SW57 SW_Push, SW58 SW_Push, SW59 SW_Push, SW60 SW_Push, SW61 SW_Push, SW62 SW_Push, SW63 SW_Push, SW64 SW_Push, SW65 SW_Push, SW66 SW_Push, SW67 SW_Push, SW68 SW_Push, SW69 SW_Push, SW70 SW_Push, SW71 SW_Push, SW72 SW_Push

Commit message: Updated pcb and projekt files.
Parts:
- SW38, SW39, SW40, SW41, SW42, SW43, SW44, SW45, SW46, SW47, SW48, SW49, SW50, SW51, SW52, SW53, SW54, SW55, SW56, SW57, SW58, SW59, SW60, SW61, SW62, SW63, SW64, SW65, SW66, SW67: footprint keyswitch:SW_Cherry_MX_1.00u_PCB -> XenophonFootprintLibrary:SW_Cherry_MX_1.00u_PCB
- SW68, SW69, SW70, SW71, SW72: footprint keyswitch:SW_Cherry_MX_1.50u_PCB -> XenophonFootprintLibrary:SW_Cherry_MX_1.50u_PCB
