File: Pro micro schematic/xenophon.sch (KiCad schematic (older format))
At the start: 4 parts, among them J1 AudioJack3, J2 AudioJack3, U1 ProMicro, U2 ProMicro

Commit message: Changed name
Changed lines of the file:
@@
 U 6107657D
 F0 "leftButtonSheet" 50
-F1 "file6107657C.sch" 50
+F1 "leftButtonSheet.sch" 50
 F2 "row1" I L 4650 2400 50
 F3 "row2" I L 4650 2500 50
@@
 U 6116737E
 F0 "rightButtonSheet" 50
-F1 "file6116737D.sch" 50
+F1 "rightButtonSheet.sch" 50
 F2 "row1" I L 9800 2500 50
 F3 "row2" I L 9800 2600 50
